File: PCB/_autosave-Shield.kicad_pcb (KiCad board)
At the start: 2 copper layers, 83.2 x 69.2 mm, 82 parts, among them J1 ADC, J10 I2C, J11 SERVO3, J12 SERVO4, J2 BATT, J3 PWR SW, J4 Screw_Terminal_01x04, J5 SERVO1, J6 ULTRA, J7 ENC1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

Commit message: Ricks Changes
Connections:
- D13 pad 2: Net-(D13-A) -> Net-(D11-A)
- D14 pad 1: Net-(D13-A) -> Net-(D11-A)
- D15 pad 2: Net-(D15-A) -> Net-(D11-A)
- D16 pad 1: Net-(D15-A) -> Net-(D11-A)
- D17 pad 2: Net-(D17-A) -> Net-(D11-A)
- D8 pad 2: Net-(D17-A) -> Net-(D11-A)
- D9 pad 1: Net-(D17-A) -> Net-(D11-A)
- J4 pad 1: Net-(D15-A) -> Net-(D11-A)
- J4 pad 2: Net-(D13-A) -> Net-(D11-A)
- J4 pad 4: Net-(D17-A) -> Net-(D11-A)
- U3 pad 16: Net-(D13-A) -> Net-(D11-A)
- U3 pad 17: Net-(D15-A) -> Net-(D11-A)
- U3 pad 4: Net-(D17-A) -> Net-(D11-A)
Routing:
- net Net-(D11-A): track 41.8 -> 158.1 mm
- net Net-(D13-A): track 41.8 -> 0.00 mm
- net Net-(D15-A): track 39.7 -> 0.00 mm
- net Net-(D17-A): track 38.9 -> 0.00 mm
